File: linefollower/board/design1.sch (EAGLE design)
At the start: 44 parts, among them IC1 STM32F10XCXT6, IC2 FT232RL, Q1 8mhz, Q2 32khz, X1 MINI-USB-32005-201

Commit message: revisi board
Parts:
- added VDD, VSS: (no value), pinhead:PINHD-1X3
Connections:
- net N$1 renamed ADC7
- net N$2 renamed ADC6
- net N$3 renamed ADC5
- net N$4 renamed ADC4
- net N$5 renamed ADC3
- net N$6 renamed ADC2
- net N$7 renamed ADC1
- net N$8 renamed ADC0
- net VDD: now also VDD.1, VDD.2, VDD.3
- net VSS: now also VSS.1, VSS.2, VSS.3
Changed lines of the file:
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@@
 <part name="C6" library="resistor" deviceset="C-EU" device="C1206" value="22pf"/>
 <part name="FRAME1" library="frames" deviceset="FRAME_A_L" device=""/>
+<part name="VDD" library="pinhead" deviceset="PINHD-1X3" device=""/>
+<part name="VSS" library="pinhead" deviceset="PINHD-1X3" device=""/>
 </parts>
 <sheets>
@@
 <instance part="FRAME1" gate="G$1" x="-43.18" y="-73.66"/>
 <instance part="FRAME1" gate="G$2" x="129.54" y="-73.66"/>
+<instance part="VDD" gate="A" x="33.02" y="-43.18" rot="R270"/>
+<instance part="VSS" gate="A" x="50.8" y="-43.18" rot="R270"/>
 </instances>
 <busses>
 </busses>
 <nets>
-<net name="N$1" class="0">
+<net name="ADC7" class="0">
 <segment>
 <pinref part="IC1" gate="PORTA_L" pin="PA7"/>
 <pinref part="PIN-ADC" gate="A" pin="1"/>
 <wire x1="43.18" y1="58.42" x2="25.4" y2="58.42" width="0.1524" layer="91"/>
-</segment>
-</net>
-<net name="N$2" class="0">
+<label x="33.02" y="58.42" size="1.778" layer="95"/>
+</segment>
+</net>
+<net name="ADC6" class="0">
 <segment>
 <pinref part="IC1" gate="PORTA_L" pin="PA6"/>
 <pinref part="PIN-ADC" gate="A" pin="2"/>
 <wire x1="43.18" y1="60.96" x2="25.4" y2="60.96" width="0.1524" layer="91"/>
-</segment>
-</net>
-<net name="N$3" class="0">
+<label x="33.02" y="60.96" size="1.778" layer="95"/>
+</segment>
+</net>
+<net name="ADC5" class="0">
 <segment>
 <pinref part="IC1" gate="PORTA_L" pin="PA5"/>
 <pinref part="PIN-ADC" gate="A" pin="3"/>
 <wire x1="43.18" y1="63.5" x2="25.4" y2="63.5" width="0.1524" layer="91"/>
-</segment>
-</net>
-<net name="N$4" class="0">
+<label x="33.02" y="63.5" size="1.778" layer="95"/>
+</segment>
+</net>
+<net name="ADC4" class="0">
 <segment>
 <pinref part="IC1" gate="PORTA_L" pin="PA4"/>
 <pinref part="PIN-ADC" gate="A" pin="4"/>
 <wire x1="43.18" y1="66.04" x2="25.4" y2="66.04" width="0.1524" layer="91"/>
-</segment>
-</net>
-<net name="N$5" class="0">
+<label x="33.02" y="66.04" size="1.778" layer="95"/>
+</segment>
+</net>
+<net name="ADC3" class="0">
 <segment>
 <pinref part="IC1" gate="PORTA_L" pin="PA3"/>
 <pinref part="PIN-ADC" gate="A" pin="5"/>
 <wire x1="43.18" y1="68.58" x2="25.4" y2="68.58" width="0.1524" layer="91"/>
-</segment>
-</net>
-<net name="N$6" class="0">
+<label x="33.02" y="68.58" size="1.778" layer="95"/>
+</segment>
+</net>
+<net name="ADC2" class="0">
 <segment>
 <pinref part="IC1" gate="PORTA_L" pin="PA2"/>
 <pinref part="PIN-ADC" gate="A" pin="6"/>
 <wire x1="43.18" y1="71.12" x2="25.4" y2="71.12" width="0.1524" layer="91"/>
-</segment>
-</net>
-<net name="N$7" class="0">
+<label x="33.02" y="71.12" size="1.778" layer="95"/>
+</segment>
+</net>
+<net name="ADC1" class="0">
 <segment>
 <pinref part="IC1" gate="PORTA_L" pin="PA1"/>
 <pinref part="PIN-ADC" gate="A" pin="7"/>
 <wire x1="43.18" y1="73.66" x2="25.4" y2="73.66" width="0.1524" layer="91"/>
-</segment>
-</net>
-<net name="N$8" class="0">
+<label x="33.02" y="73.66" size="1.778" layer="95"/>
+</segment>
+</net>
+<net name="ADC0" class="0">
 <segment>
 <pinref part="IC1" gate="PORTA_L" pin="PA0"/>
 <pinref part="PIN-ADC" gate="A" pin="8"/>
 <wire x1="43.18" y1="76.2" x2="25.4" y2="76.2" width="0.1524" layer="91"/>
+<label x="33.02" y="76.2" size="1.778" layer="95"/>
 </segment>
 </net>
@@
 <label x="205.74" y="15.24" size="1.778" layer="95"/>
 </segment>
+<segment>
+<pinref part="VDD" gate="A" pin="3"/>
+<wire x1="30.48" y1="-40.64" x2="30.48" y2="-30.48" width="0.1524" layer="91"/>
+<wire x1="30.48" y1="-30.48" x2="33.02" y2="-30.48" width="0.1524" layer="91"/>
+<pinref part="VDD" gate="A" pin="1"/>
+<wire x1="33.02" y1="-30.48" x2="35.56" y2="-30.48" width="0.1524" layer="91"/>
+<wire x1="35.56" y1="-30.48" x2="35.56" y2="-40.64" width="0.1524" layer="91"/>
+<pinref part="VDD" gate="A" pin="2"/>
+<wire x1="33.02" y1="-40.64" x2="33.02" y2="-30.48" width="0.1524" layer="91"/>
+<label x="35.56" y="-30.48" size="1.778" layer="95"/>
+</segment>
 </net>
 <net name="VSS" class="0">
@@
 <label x="167.64" y="12.7" size="1.778" layer="95"/>
 </segment>
-</net>
+<segment>
+<pinref part="VSS" gate="A" pin="3"/>
+<wire x1="48.26" y1="-40.64" x2="48.26" y2="-30.48" width="0.1524" layer="91"/>
+<wire x1="48.26" y1="-30.48" x2="50.8" y2="-30.48" width="0.1524" layer="91"/>
+<pinref part="VSS" gate="A" pin="1"/>
+<wire x1="50.8" y1="-30.48" x2="53.34" y2="-30.48" width="0.1524" layer="91"/>
+<wire x1="53.34" y1="-30.48" x2="53.34" y2="-40.64" width="0.1524" layer="91"/>
+<pinref part="VSS" gate="A" pin="2"/>
+<wire x1="50.8" y1="-40.64" x2="50.8" y2="-30.48" width="0.1524" layer="91"/>
+<label x="53.34" y="-30.48" size="1.778" layer="95"/>
+</segment>
+</net>
